File: hardware/ElectricalCabinet/ElectricalCabinet/ElectricalCabinet.kicad_sch (KiCad schematic)
At the start: 19 parts

Commit message: Updates on Cabinet
Connections:
- net 110-1 renamed 6110-1
- net 110-11 renamed 6110-11
- net 110-13 renamed 6110-13
- net 110-15 renamed 6110-15
- net 110-17 renamed 6110-17
- net 110-19 renamed 6110-19
- net 110-21 renamed 6110-21
- net 110-23 renamed 6110-23
- net 110-25 renamed 6110-25
- net 110-27 renamed 6110-27
- net 110-29 renamed 6110-29
- net 110-31 renamed 6110-31
- net 110-33 renamed 6110-33
- net 110-35 renamed 6110-35
- net 110-37 renamed 6110-37
- net 110-5 renamed 6110-5
- net 110-7 renamed 6110-7
- net 110-9 renamed 6110-9
Other:
- sheet 6110Block (page 23) renamed 6110Block
- sheet 5000Block: file 500Block.kicad_sch -> 5000Block.kicad_sch
- sheet 5500Block: file 550Block.kicad_sch -> 5500Block.kicad_sch
- sheet 6100Block: file 100Block.kicad_sch -> 6100Block.kicad_sch
- sheet 6110Block: file 110Block.kicad_sch -> 6110Block.kicad_sch
