File: hardware/ElectricalCabinet/ElectricalCabinet/ElectricalCabinet.kicad_sch (KiCad schematic)
At the start: 19 parts

Commit message: Further wiring updates
Populated 6100 Bus
Corrected number of relay boards
Added 110v outputs to relay boards and noted light positon
Uploaded light scheme to documents folder
Parts:
- removed F14, F15, F16, F17, F18, F19: 2.5A, symbol PCM_Device_AKL:Fuse
Other:
- removed sheet 8100Block
- removed sheet RelayBoard12
- removed sheet RelayBoard13
- removed sheet RelayBoard14
- removed sheet RelayBoard15
- removed sheet RelayBoard16
- removed sheet RelayBoard17

Commit message: Electrical Cabinet done
Electrical Cabinet done, let me know if there are any changes or mistakes.
Other:
- removed sheet 6110Block
Changed lines of the file:
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@@
 		(property "Ref" "Ref 2100"
 			(at 93.726 41.91 0)
+			(hide yes)
 			(show_name no)
 			(do_not_autoplace no)
@@
 		(property "Ref" "Ref 2000"
 			(at 93.726 48.26 0)
+			(hide yes)
 			(show_name no)
 			(do_not_autoplace no)
@@
 		(property "Ref" "Ref 108"
 			(at 71.12 43.18 0)
+			(hide yes)
 			(show_name no)
 			(do_not_autoplace no)
@@
 				)
 			)
-		)
-	)
-	(sheet
-		(at 153.67 133.35)
-		(size 12.7 3.81)
-		(exclude_from_sim no)
-		(in_bom yes)
-		(on_board yes)
-		(dnp no)
-		(fields_autoplaced yes)
-		(stroke
-			(width 0.1524)
-			(type solid)
-		)
-		(fill
-			(color 0 0 0 0)
-		)
-		(property "Sheetname" "6110Block"
-			(at 153.67 132.6384 0)
-			(show_name no)
-			(do_not_autoplace no)
-			(effects
-				(font
-					(size 1.27 1.27)
-				)
-				(justify left bottom)
-			)
-		)
-		(property "Sheetfile" "6110Block.kicad_sch"
-			(at 153.67 137.7446 0)
-			(show_name no)
-			(do_not_autoplace no)
-			(effects
-				(font
-					(size 1.27 1.27)
-				)
-				(justify left top)
-			)
-		)
-		(instances
-			(project "ElectricalCabinet"
-				(path "/c34866b5-fe82-42ea-9d09-ac7e183279a1"
-					(page "23")
-				)
-			)
