File: hardware/ElectricalCabinet/ElectricalCabinet/6100Block.kicad_sch (KiCad schematic)
At the start: 0 parts

Commit message: Further wiring updates
Populated 6100 Bus
Corrected number of relay boards
Added 110v outputs to relay boards and noted light positon
Uploaded light scheme to documents folder
Parts:
- added U13, U14, U15, U16, U17, U18, U19, U20, U21, U22, U23, U24, U25, U26, U27, U28, U29, U30, U31, U32, U33, U34, U35, U36, U37, U38, U39, U40, U41, U42, U43, U44, U45, U46, U47, U48, U49, U50, U51, U52, U53, U54, U55, U56, U57: (no value), symbol TrafficLightLibrary:Terminal_Block
Connections:
- new net: U13. (2), U14. (2), U15. (2), U16. (2), U17. (2), U18. (2), U19. (2), U20. (2), U21. (2), U22. (2), U23. (2), U24. (2), U25. (2), U26. (2), U27. (2), U28. (2), U29. (2), U30. (2), U31. (2), U32. (2), U33. (2), U34. (2), U35. (2), U36. (2), U37. (2), U38. (2), U39. (2), U40. (2), U41. (2), U42. (2), U43. (2), U44. (2), U45. (2), U46. (2), U47. (2), U48. (2), U49. (2), U50. (2), U51. (2), U52. (2), U53. (2), U54. (2), U55. (2), U56. (2), U57. (2)
- new net 6100-1: U13. (2)
- new net 6100-10: U22. (2)
- new net 6100-11: U23. (2)
- new net 6100-12: U24. (2)
- new net 6100-13: U25. (2)
- new net 6100-14: U26. (2)
- new net 6100-15: U27. (2)
- new net 6100-16: U28. (2)
- new net 6100-17: U29. (2)
- new net 6100-18: U30. (2)
- new net 6100-19: U31. (2)
- new net 6100-2: U14. (2)
- new net 6100-20: U32. (2)
- new net 6100-21: U33. (2)
- new net 6100-22: U34. (2)
- new net 6100-23: U35. (2)
- new net 6100-24: U36. (2)
- new net 6100-25: U37. (2)
- new net 6100-26: U38. (2)
- new net 6100-27: U39. (2)
- new net 6100-28: U40. (2)
- new net 6100-29: U41. (2)
- new net 6100-3: U15. (2)
- new net 6100-30: U42. (2)
- new net 6100-31: U43. (2)
- new net 6100-32: U44. (2)
- new net 6100-33: U45. (2)
- new net 6100-34: U46. (2)
- new net 6100-35: U47. (2)
- new net 6100-36: U48. (2)
- new net 6100-37: U49. (2)
- new net 6100-38: U50. (2)
- new net 6100-39: U51. (2)
- new net 6100-4: U16. (2)
- new net 6100-40: U52. (2)
- new net 6100-41: U53. (2)
- new net 6100-42: U54. (2)
- new net 6100-43: U55. (2)
- new net 6100-44: U56. (2)
- new net 6100-45: U13. (2)
- new net 6100-46: U14. (2)
- new net 6100-47: U15. (2)
- new net 6100-48: U16. (2)
- new net 6100-49: U17. (2)
- new net 6100-5: U17. (2)
- new net 6100-50: U18. (2)
- new net 6100-51: U19. (2)
- new net 6100-52: U20. (2)
- new net 6100-53: U21. (2)
- new net 6100-54: U22. (2)
- new net 6100-55: U23. (2)
- new net 6100-56: U24. (2)
- new net 6100-57: U25. (2)
- new net 6100-58: U26. (2)
- new net 6100-59: U27. (2)
- new net 6100-6: U18. (2)
- new net 6100-60: U28. (2)
- new net 6100-61: U29. (2)
- new net 6100-62: U30. (2)
- new net 6100-63: U31. (2)
- new net 6100-64: U32. (2)
- new net 6100-65: U33. (2)
- new net 6100-66: U34. (2)
- new net 6100-67: U35. (2)
- new net 6100-68: U36. (2)
- new net 6100-69: U37. (2)
- new net 6100-7: U19. (2)
- new net 6100-70: U38. (2)
- new net 6100-71: U39. (2)
- new net 6100-72: U40. (2)
- new net 6100-73: U41. (2)
- new net 6100-74: U42. (2)
- new net 6100-75: U43. (2)
- new net 6100-76: U44. (2)
- new net 6100-77: U45. (2)
- new net 6100-78: U46. (2)
- new net 6100-79: U47. (2)
- new net 6100-8: U20. (2)
- new net 6100-80: U48. (2)
- new net 6100-81: U49. (2)
- new net 6100-82: U50. (2)
- new net 6100-83: U51. (2)
- new net 6100-84: U52. (2)
- new net 6100-85: U53. (2)
- new net 6100-86: U54. (2)
- new net 6100-87: U55. (2)
- new net 6100-88: U56. (2)
- new net 6100-9: U21. (2)
- new net 6100-99: U57. (2)
