File: hardware/ElectricalCabinet/ElectricalCabinet/2_ControlBoard.kicad_sch (KiCad schematic)
At the start: 0 parts

Commit message: Cabinet Schematics Update
Parts:
- added 1000BLOCK1: SN74AHCT125N, N14, symbol 2026-07-22_17-51-08:SN74AHCT125N
- added J3: Screw_Terminal_01x06, symbol Connector:Screw_Terminal_01x06
- added U1: ESP32-DevKitC, PCM_Espressif:ESP32-DevKitC, symbol PCM_Espressif:ESP32-DevKitC
Connections:
- new net 3.3V Clock In: 1000BLOCK1.2 (1A), U1.30 (GPIO18)
- new net 3.3V Data In: 1000BLOCK1.9 (3A), U1.37 (GPIO23)
- new net 3.3V Enable In: 1000BLOCK1.12 (4A), U1.26 (ADC2_CH0/GPIO4)
- new net 3.3V Latch In: 1000BLOCK1.5 (2A), U1.29 (GPIO5)
- new net 5V Clock Out: 1000BLOCK1.3 (1Y), J3.3 (Pin_3)
- new net 5V Enable Out: 1000BLOCK1.11 (4Y), J3.1 (Pin_1)
- new net 5V GND: 1000BLOCK1.1 (*1OE), 1000BLOCK1.10 (*3OE), 1000BLOCK1.13 (*4OE), 1000BLOCK1.4 (*2OE), 1000BLOCK1.7 (GND), J3.5 (Pin_5), U1.14 (GND), U1.32 (GND), U1.38 (GND)
- new net 5V Latch Out: 1000BLOCK1.6 (2Y), J3.2 (Pin_2)
- new net 5V Power: 1000BLOCK1.14 (VCC), J3.6 (Pin_6), U1.19 (5V)
- new net Serial Out: 1000BLOCK1.8 (3Y), J3.4 (Pin_4)
