File: hardware/ElectricalCabinet/ElectricalCabinet/8200Block.kicad_sch (KiCad schematic)
At the start: 0 parts

Commit message: Electrical Cabinet done
Electrical Cabinet done, let me know if there are any changes or mistakes.
Parts:
- added U58, U59, U60, U61, U62, U63: (no value), symbol TrafficLightLibrary:Terminal_Block
Connections:
- net 8200-1: now also U58. (2)
- net 8200-2: now also U59. (2)
- new net: U58. (2), U59. (2), U60. (2), U61. (2), U62. (2), U63. (2)
- new net 8200-10: U60. (2)
- new net 8200-11: U59. (2)
- new net 8200-12: U58. (2)
- new net 8200-3: U60. (2)
- new net 8200-4: U61. (2)
- new net 8200-5: U62. (2)
- new net 8200-6: U63. (2)
- new net 8200-7: U63. (2)
- new net 8200-8: U62. (2)
- new net 8200-9: U61. (2)
