File: hardware/MainBoard/TrafficLight.kicad_sch (KiCad schematic)
At the start: 3 parts, among them J3 Screw_Terminal_01x06, U1 ESP32-DevKitC

Commit message: Updates on Cabinet
Connections:
- net 5V Clock Out: now reaches 1000BLOCK.3 (1Y)
- net 5V Clock Out: now also J3.3 (Pin_3); no longer J3.1 (Pin_1)
- net 5V GND: now reaches 1000BLOCK.7 (GND), U1.14 (GND), U1.32 (GND), U1.38 (GND)
- net 5V GND: now also 1000BLOCK.1 (*1OE), 1000BLOCK.10 (*3OE), 1000BLOCK.13 (*4OE), 1000BLOCK.4 (*2OE), J3.5 (Pin_5); no longer J3.2 (Pin_2)
- net 5V Latch Out: now reaches 1000BLOCK.6 (2Y)
- net 5V Latch Out: now also J3.2 (Pin_2); no longer J3.3 (Pin_3)
- net 5V Power: now reaches 1000BLOCK.14 (VCC), U1.19 (5V)
- net 5V Power: now also J3.6 (Pin_6); no longer J3.4 (Pin_4)
- net Serial Out: now reaches 1000BLOCK.8 (3Y)
- net Serial Out: now also J3.4 (Pin_4); no longer J3.6 (Pin_6)
- net at U1.27 (GPIO16): no longer 1000BLOCK.11 (4Y)
- net 3.3V Enable In: now reaches 1000BLOCK.12 (4A)
- net 3.3V Enable In: now also U1.26 (ADC2_CH0/GPIO4)
- net 3.3V Clock In: now reaches 1000BLOCK.2 (1A)
- net 3.3V Clock In: now also U1.30 (GPIO18); no longer U1.37 (GPIO23)
- net 3.3V Latch In: now reaches 1000BLOCK.5 (2A)
- net 3.3V Latch In: now also U1.29 (GPIO5); no longer U1.30 (GPIO18)
- net 3.3V Data In: now reaches 1000BLOCK.9 (3A)
- net 3.3V Data In: now also U1.37 (GPIO23); no longer U1.29 (GPIO5)
- new net 5V Enable Out: 1000BLOCK.11 (4Y), J3.1 (Pin_1)
Other:
- note removed: "1000-10"
- note removed: "1000-3"
- note removed: "1000-6"
- note removed: "1000-8"
- note removed: "500-1"
- note removed: "550-1"

Commit message: Cabinet Schematics Update
Other:
- note added: "5000-2"
- note added: "5500-2"
- note added: "7500-1"
- note added: "8100-1"
- note added: "8200-1"
- note added: "8300-1"
Changed lines of the file:
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@@
 		(date "2026-07-22")
+	)
+	(text "5500-2"
+		(exclude_from_sim no)
+		(at 211.074 48.768 90)
+		(effects
+			(font
+				(size 1.27 1.27)
+			)
+		)
+	)
+	(text "5000-2"
+		(exclude_from_sim no)
+		(at 208.534 48.768 90)
+		(effects
+			(font
+				(size 1.27 1.27)
+			)
+		)
+	)
+	(text "7500-1"
+		(exclude_from_sim no)
+		(at 205.994 48.768 90)
+		(effects
+			(font
+				(size 1.27 1.27)
+			)
+		)
+	)
+	(text "8200-1"
+		(exclude_from_sim no)
+		(at 200.914 48.768 90)
+		(effects
+			(font
+				(size 1.27 1.27)
+			)
+		)
+	)
+	(text "8100-1"
+		(exclude_from_sim no)
+		(at 198.374 48.768 90)
+		(effects
+			(font
+				(size 1.27 1.27)
+			)
+		)
+	)
+	(text "8300-1"
+		(exclude_from_sim no)
+		(at 203.454 48.768 90)
+		(effects
+			(font
+				(size 1.27 1.27)
+			)
+		)
 	)
 	(junction
