File: hardware/RelayBoard/TrafficLight_RelayModule.kicad_pcb (KiCad board)
At the start: 2 copper layers, 76 x 76 mm, 28 parts, among them J1 Screw_Terminal_01x09, J2 Screw_Terminal_01x06, K1 G3MB-202P DC5, K2 G3MB-202P DC5, K3 G3MB-202P DC5, K4 G3MB-202P DC5, K5 G3MB-202P DC5, K6 G3MB-202P DC5, K7 G3MB-202P DC5, K8 G3MB-202P DC5, U1 TPIC6B595N

Commit message: Updates to electrical board after review
Parts:
- moved K5 25.6 mm to (59.6, 34.9)
- moved D5 24.0 mm to (61.0, 59.7)
- moved R5 24.0 mm to (61.0, 62.2)
- moved D8 22.9 mm to (38.1, 59.7)
- moved R8 22.9 mm to (38.1, 62.2)
- moved K8 21.3 mm to (36.7, 34.9)
- moved K6 9.94 mm to (51.9, 34.9)
- moved D6 8.35 mm to (53.3, 59.7)
- moved R6 8.34 mm to (53.3, 62.2)
- moved D7 7.29 mm to (45.7, 59.7)
- moved R7 7.29 mm to (45.7, 62.2)
- moved K7 5.68 mm to (44.3, 34.9)
- moved D1 1.59 mm to (91.4, 59.7)
- moved R1 1.58 mm to (91.4, 62.2)
- moved D2 1.22 mm to (83.8, 59.7)
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Connections:
- C1 pad 1: Net-(J2-Pin_2) -> +5V
- C1 pad 2: Net-(J2-Pin_6) -> GND
- D1 pad 2: Net-(D1-A) -> +5V
- D2 pad 2: Net-(D1-A) -> +5V
- D3 pad 2: Net-(D1-A) -> +5V
- D4 pad 2: Net-(D1-A) -> +5V
- D5 pad 2: Net-(D1-A) -> +5V
- D6 pad 2: Net-(D1-A) -> +5V
- D7 pad 2: Net-(D1-A) -> +5V
- D8 pad 2: Net-(D1-A) -> +5V
- J1 pad 9: Net-(J1-Pin_9) -> /110vAC Hawt
- J2 pad 1: Net-(J2-Pin_1) -> GND
- J2 pad 6: Net-(J2-Pin_6) -> +5V
- K1 pad 1: Net-(J1-Pin_9) -> Net-(J1-Pin_1)
- K1 pad 2: Net-(J1-Pin_1) -> /110vAC Hawt
- K1 pad 3: Net-(D1-A) -> +5V
- K2 pad 1: Net-(J1-Pin_9) -> Net-(J1-Pin_2)
- K2 pad 2: Net-(J1-Pin_2) -> /110vAC Hawt
- K2 pad 3: Net-(D1-A) -> +5V
- K3 pad 1: Net-(J1-Pin_9) -> Net-(J1-Pin_3)
- K3 pad 2: Net-(J1-Pin_3) -> /110vAC Hawt
- K3 pad 3: Net-(D1-A) -> +5V
- K4 pad 1: Net-(J1-Pin_9) -> Net-(J1-Pin_4)
- K4 pad 2: Net-(J1-Pin_4) -> /110vAC Hawt
- K4 pad 3: Net-(D1-A) -> +5V
- K5 pad 1: Net-(J1-Pin_9) -> Net-(J1-Pin_5)
- K5 pad 2: Net-(J1-Pin_5) -> /110vAC Hawt
- K5 pad 3: Net-(D1-A) -> +5V
- K6 pad 1: Net-(J1-Pin_9) -> Net-(J1-Pin_6)
- K6 pad 2: Net-(J1-Pin_6) -> /110vAC Hawt
- K6 pad 3: Net-(D1-A) -> +5V
- K7 pad 1: Net-(J1-Pin_9) -> Net-(J1-Pin_7)
- K7 pad 2: Net-(J1-Pin_7) -> /110vAC Hawt
- K7 pad 3: Net-(D1-A) -> +5V
- K8 pad 1: Net-(J1-Pin_9) -> Net-(J1-Pin_8)
- K8 pad 2: Net-(J1-Pin_8) -> /110vAC Hawt
- K8 pad 3: Net-(D1-A) -> +5V
- U1 pad 10: Net-(J2-Pin_2) -> GND
- U1 pad 11: Net-(J2-Pin_2) -> GND
- U1 pad 12: Net-(J2-Pin_4) -> Net-(J2-Pin_2)
- U1 pad 18: Net-(J2-Pin_1) -> Net-(J2-Pin_4)
- U1 pad 19: Net-(J2-Pin_2) -> GND
- U1 pad 2: Net-(J2-Pin_6) -> +5V
- U1 pad 8: Net-(J2-Pin_6) -> +5V
- U1 pad 9: Net-(J2-Pin_2) -> GND
Routing:
- net +5V: track 0.00 -> 187.7 mm
- net Net-(J1-Pin_9): track 164.5 -> 0.00 mm
- net Net-(D1-A): track 115.6 -> 0.00 mm
- net /110vAC Hawt: track 0.00 -> 85.2 mm
- net Net-(J2-Pin_2): track 84.3 -> 10.4 mm
- net Net-(J2-Pin_6): track 37.0 -> 0.00 mm
- net Net-(J1-Pin_5): track 48.3 -> 12.1 mm
- net Net-(J1-Pin_8): track 49.9 -> 15.3 mm
- net Net-(J2-Pin_1): track 33.7 -> 0.00 mm
- net Net-(U1-DRAIN4): track 64.7 -> 36.1 mm, vias 0 -> 1
- net Net-(J2-Pin_5): track 40.6 -> 18.3 mm
- net Net-(J1-Pin_7): track 35.1 -> 14.2 mm
- net Net-(U1-DRAIN7): track 48.3 -> 64.3 mm, vias 0 -> 1
- net Net-(U1-DRAIN5): track 59.3 -> 45.5 mm, vias 0 -> 1
- net Net-(J1-Pin_6): track 26.3 -> 13.2 mm
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- added copper zone on B.Cu, net GND
Other:
- board size 76 x 76 mm -> 76 x 78.8 mm
- board text added: "+5V"
- board text added: "110VAC HOT"
- board text added: "CH1"
- board text added: "CH2"
- board text added: "CH3"
- board text added: "CH4"
- board text added: "CH5"
- board text added: "CH6"
- board text added: "CH7"
- board text added: "CH8"
- board text added: "CLK"
- board text added: "GND"
- board text added: "IN"
- board text added: "LOAD"
- board text added: "OUT"
- board text added: "TPIC6B595N"
- board text added: "Traffic Light Clock Relay Board Copyright (C) Boden Research 2026 Designed by: ghrrum Assisted by: MadManMarkAu"
- board text added: "U1"
