File: hardware/RelayBoard/TrafficLight_RelayModule.kicad_sch (KiCad schematic)
At the start: 28 parts, among them J1 Screw_Terminal_01x09, J2 Screw_Terminal_01x06, K1 G3MB-202P DC5, K2 G3MB-202P DC5, K3 G3MB-202P DC5, K4 G3MB-202P DC5, K5 G3MB-202P DC5, K6 G3MB-202P DC5, K7 G3MB-202P DC5, K8 G3MB-202P DC5, U1 TPIC6B595N

Commit message: Cabinet Schematics Update
Other:
- moved on the sheet: C1, U1

Commit message: Updates to electrical board after review
Connections:
- net 110vAC Hawt: now also K1.2, K2.2, K3.2, K4.2, K5.2, K6.2, K7.2, K8.2; no longer K1.1, K2.1, K3.1, K4.1, K5.1, K6.1, K7.1, K8.1
- net at J1.8 (Pin_8): now also K8.1; no longer K8.2
- net +5V: now reaches D1.2 (A), D2.2 (A), D3.2 (A), D4.2 (A), D5.2 (A), D6.2 (A), D7.2 (A), D8.2 (A), K1.3, K2.3, K3.3, K4.3, K5.3, K6.3, K7.3, K8.3
- net +5V: now also C1.1, J2.6 (Pin_6), U1.2 (VCC), U1.8 (~{SRCLR})
- net at J1.3 (Pin_3): now also K3.1; no longer K3.2
- net at J1.4 (Pin_4): now also K4.1; no longer K4.2
- net at J1.6 (Pin_6): now also K6.1; no longer K6.2
- net at J1.5 (Pin_5): now also K5.1; no longer K5.2
- net at J1.1 (Pin_1): now also K1.1; no longer K1.2
- net at J1.2 (Pin_2): now also K2.1; no longer K2.2
- net at J1.7 (Pin_7): now also K7.1; no longer K7.2
- net GND: now reaches U1.10 (GND), U1.11 (GND), U1.19 (GND), U1.9 (~{G})
- net GND: now also C1.2, J2.1 (Pin_1); no longer C1.1, J2.2 (Pin_2)
- net at U1.12 (RCK): now also J2.2 (Pin_2); no longer J2.4 (Pin_4)
- net at U1.18 (SEROUT): now also J2.4 (Pin_4); no longer J2.1 (Pin_1)
Other:
- note added: "+5V"
- note added: "CLK"
- note added: "GND"
- note added: "IN"
- note added: "LOAD"
- note added: "OUT"
- note removed: "1000-3"
- note removed: "1000-6"
- note removed: "1000-8"
- note removed: "500-1"
- note removed: "550-1"
- note removed: "7400-1"
- moved on the sheet: C1
